File: mcu board redesign/kicad/Kunlun STM32 MCU Board.kicad_pcb (KiCad board)
At the start: 2 copper layers, 40 x 40 mm, 40 parts, among them J1 0532610671, J2 10129383-908001ALF, J3 USB4105-GF-A, J4 5002, J5 5002, J6 5002, J7 5002, J8 5001, J9 5001, SW1 KMR231NG ULC LFS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

Commit message: Set rev to 1a
It was set to 2 but there were other changes planned that I didn't keep.
Other:
- board text added: "Kunlun STM32 MCU Board r1a"
- board text removed: "Kunlun STM32 MCU Board r2"
Changed lines of the file:
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@@
 		)
 	)
-	(gr_text "Kunlun STM32 MCU Board r2"
-		(at 153.5 92.5 0)
+	(gr_text "Kunlun STM32 MCU Board r1a"
+		(at 153 92.5 0)
 		(layer "B.SilkS")
 		(effects
